File: TalTechHeat.kicad_sch (KiCad schematic)
At the start: 76 parts, among them J1 02x03, J2 OLED_SSD1306, J3 XT-30, J4 Conn_01x04, Q1 DMP4015SPSQ-13, Q2 PJQ4439EP-AU_R2_002A1, Q3 PJQ4439EP-AU_R2_002A1, Q4 IRLR8726TRPBF, Q5 SS8050-G, SW1 Reset_Switch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

Commit message: Updated new parts MFN and MPN as well as title block
Parts:
- J4: MFN (none) -> JST Commercial; MPN (none) -> B4B-PH-K-S(LF)(SN); Mouser_PN (none) -> 306-B4BPHKSLFSNPP
Changed lines of the file:
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@@
 	(title_block
 		(title "Reflow Plate")
-		(date "2026-01-10")
-		(rev "1.3")
+		(date "2026-01-16")
+		(rev "1.4")
 		(company "Taltech")
 		(comment 1 "Robin Madar")
@@
 			)
 		)
+		(property "S1PN" ""
+			(at 311.15 220.98 0)
+			(effects
+				(font
+					(size 1.27 1.27)
+				)
+				(hide yes)
+			)
+		)
+		(property "S1PL" ""
+			(at 311.15 220.98 0)
+			(effects
+				(font
+					(size 1.27 1.27)
+				)
+				(hide yes)
+			)
+		)
+		(property "S1SN" ""
+			(at 311.15 220.98 0)
+			(effects
+				(font
+					(size 1.27 1.27)
+				)
+				(hide yes)
+			)
+		)
+		(property "MFN" "JST Commercial "
+			(at 311.15 220.98 0)
+			(effects
+				(font
+					(size 1.27 1.27)
+				)
+				(hide yes)
+			)
+		)
+		(property "MPN" " B4B-PH-K-S(LF)(SN) "
+			(at 311.15 220.98 0)
+			(effects
+				(font
+					(size 1.27 1.27)
+				)
+				(hide yes)
+			)
+		)
+		(property "Mouser_PN" " 306-B4BPHKSLFSNPP "
+			(at 311.15 220.98 0)
+			(effects
+				(font
+					(size 1.27 1.27)
+				)
+				(hide yes)
+			)
+		)
 		(pin "3"
 		)
@@
 			(at 266.7 209.55 0)
 			(effects
+				(font
+					(size 1.27 1.27)
+				)
+				(hide yes)
+			)
+		)
+		(property "S1PN" ""
+			(at 266.7 209.55 0)
+			(effects
+				(font
+					(size 1.27 1.27)
+				)
+				(hide yes)
+			)
+		)
+		(property "S1PL" ""
+			(at 266.7 209.55 0)
+			(effects
+				(font
+					(size 1.27 1.27)
+				)
+				(hide yes)
+			)
+		)
+		(property "S1SN" ""
+			(at 266.7 209.55 0)
+			(effects

Commit message: ReadMe
Parts:
- added U5: (no value), AA:SOP-8_CH340N, symbol AA:CH340N
Connections:
- net BUT1: now also U1.2 (PC13)
- net BUT2: now also U1.3 (PC14)
- net D_N: now also U5.2 (UD-); no longer U1.32 (PA11)
- net D_P: now also U5.1 (UD+); no longer U1.33 (PA12)
- net GND: now also U5.3 (GND)
- net PWM: now also U1.26 (PB13); no longer U1.43 (PB7)
- net VCC-DIV: now also U1.13 (PA3); no longer U1.30 (PA9)
- net PC15: now reaches J1.1 (Pin_1)
- net PC15: now also U1.4 (PC15)
- net UART1_TX: now reaches U1.31 (PA10)
- net UART1_TX: now also U5.6 (TXD)
- net SWDIO: now reaches U1.34 (PA13)
- net SWDIO: now also J1.3 (Pin_3)
- net SWCLK: now reaches U1.37 (PA14)
- net SWCLK: now also J1.5 (Pin_5)
- removed net UART2_RX: J1.5 (Pin_5), U1.13 (PA3)
- net UART2_TX: no longer names the net of U1.12 (PA2)
- net UART2_TX: no longer J1.3 (Pin_3)
- new net UART1_RX: U1.30 (PA9), U5.7 (RXD)
- no-connect marks 26 -> 21

Commit message: Fixes implementation 1/2
Parts:
- added C27, C28: 100nF, Capacitor_SMD:C_0603_1608Metric_Pad1.08x0.95mm_HandSolder, symbol Device:C
- U5: footprint AA:SOP-8_CH340N -> Package_SO:SOP-8_3.76x4.96mm_P1.27mm
Connections:
- net +3.3V: now also U5.5 (VCC), C27.1
- net GND: now also C27.2, C28.2
- net NRST: now also U5.4 (RST#)
- net TEMP_1: now also J4.3 (Pin_3); no longer J4.2 (Pin_2)
- net TEMP_2: now also J4.2 (Pin_2); no longer J4.3 (Pin_3)
- net at U5.8 (V3): now also C28.1
- no-connect marks 21 -> 22
Other:
- note added: "CH340N"
- moved on the sheet: C10, C11, C19, C20, C21, C22, C23, C24, C5, C6, C7, C8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
